Commit message: ur works

File: ur_linear_guide/urdf/linear_ur.urdf.xacro (robot description, xacro)
@@ -12,5 +12,5 @@
     <!-- ur -->
     <xacro:property name="ur_type" value="ur5"/>
-    <xacro:property name="name" value="ur"/>
+    <xacro:property name="name" value="ur5"/>
     <xacro:property name="tf_prefix" value=""/>
     <xacro:property name="joint_limit_params" value="$(find ur_linear_guide)/config/ur5/joint_limits.yaml"/>
@@ -25,8 +25,8 @@
     <xacro:property name="safety_k_position" value="20"/>
     <xacro:property name="headless_mode" value="false"/>
-    <xacro:property name="robot_ip" value="0.0.0.0"/>
-    <xacro:property name="script_filename" value=""/>
-    <xacro:property name="output_recipe_filename" value=""/>
-    <xacro:property name="input_recipe_filename" value=""/>
+    <xacro:property name="robot_ip" value="192.168.1.102"/>
+    <xacro:property name="script_filename" value="$(find ur_client_library)/resources/external_control.urscript"/>
+    <xacro:property name="input_recipe_filename" value="$(find ur_robot_driver)/resources/rtde_input_recipe.txt"/>
+    <xacro:property name="output_recipe_filename" value="$(find ur_robot_driver)/resources/rtde_output_recipe.txt"/>
     <xacro:property name="reverse_ip" value="0.0.0.0"/>
     <xacro:property name="script_command_port" value="50004"/>

File: ur_linear_guide/urdf/linear_ur.xacro (robot description, xacro)
@@ -10,5 +10,5 @@
     vel_lim:=0.5
     ur_type:=ur5
-    name:=ur
+    name:=ur5
     tf_prefix:=''
     joint_limits_parameters_file:='$(find ur_description)/config/ur5/joint_limits.yaml'
@@ -35,5 +35,5 @@
     tool_device_name:=/tmp/ttyUR
     tool_tcp_port:=54321
-    robot_ip:=0.0.0.0
+    robot_ip:=192.168.1.102
     script_filename:=to_be_filled_by_ur_robot_driver
     output_recipe_filename:=to_be_filled_by_ur_robot_driver

Commit message: works

File: ur_linear_guide/urdf/linear_ur.urdf.xacro (robot description, xacro)
@@ -4,4 +4,5 @@
     <xacro:arg name="fake_guide" default="true"/>
     <xacro:arg name="fake_ur" default="true"/>
+    <xacro:arg name="fake_robotiq" default="true"/>
     <!-- properties -->
     <!-- linear guide -->
@@ -99,3 +100,8 @@
       keep_alive_count="${keep_alive_count}"
     />
+  <!-- robotiq gripper -->
+  <xacro:include filename="$(find robotiq_description)/urdf/robotiq_2f_85_macro.urdf.xacro" />
+  <xacro:robotiq_gripper name="RobotiqGripperHardwareInterface" prefix="" parent="tool0" use_fake_hardware="$(arg fake_robotiq)" include_ros2_control="true" com_port="/dev/ttyUSB1">
+      <origin xyz="0 0 0" rpy="0 0 0" />
+  </xacro:robotiq_gripper>
 </robot>
