Commit message: fix

File: ur_linear_guide/urdf/linear_guide.xacro (robot description, xacro)
@@ -44,5 +44,5 @@
     <parent link = "guide_base_link"/>
     <child link = "guide_link"/>
-    <origin xyz = "${-length/2} 0.0 0.0"/>
+    <origin xyz = "${length/2 - max_lim} 0.0 0.0"/>
     <limit effort="1000.0" lower="${min_lim}" upper="${max_lim}" velocity="${vel_lim}"/>
     <axis xyz = "1 0 0"/>

File: ur_linear_guide/urdf/linear_ur.urdf.xacro (robot description, xacro)
@@ -1,50 +1,53 @@
 <?xml version="1.0" encoding="utf-8"?>
 <robot xmlns:xacro="http://www.ros.org/wiki/xacro" name="ur_on_linear_guide">
+    <!-- args -->
     <xacro:arg name="fake_guide" default="true"/>
     <xacro:arg name="fake_ur" default="true"/>
-    <xacro:arg name="length" default="1.56"/>
-    <xacro:arg name="min_lim" default="0.05"/>
-    <xacro:arg name="max_lim" default="1.50"/>
-    <xacro:arg name="vel_lim" default="0.5"/>
-    <xacro:arg name="ur_type" default="ur5"/>
-    <xacro:arg name="name" default="ur"/>
-    <xacro:arg name="tf_prefix" default=""/>
-    <xacro:arg name="joint_limit_params" default="$(find ur_linear_guide)/urdf/joint_limits.yaml"/>
-    <xacro:arg name="kinematics_params" default="$(find ur_linear_guide)/urdf/default_kinematics.yaml"/>
-    <xacro:arg name="physical_params" default="$(find ur_linear_guide)/urdf/physical_parameters.yaml"/>
-    <xacro:arg name="visual_params" default="$(find ur_linear_guide)/urdf/visual_parameters.yaml"/>
-    <xacro:arg name="initial_positions_file" default="$(find ur_linear_guide)/urdf/initial_positions.yaml"/>
-    <xacro:arg name="transmission_hw_interface" default=""/>
-    <xacro:arg name="safety_limits" default="false"/>
-    <xacro:arg name="safety_pos_margin" default="0.15"/>
-    <xacro:arg name="safety_k_position" default="20"/>
-    <xacro:arg name="headless_mode" default="false"/>
-    <xacro:arg name="robot_ip" default="0.0.0.0"/>
-    <xacro:arg name="script_filename" default=""/>
-    <xacro:arg name="output_recipe_filename" default=""/>
-    <xacro:arg name="input_recipe_filename" default=""/>
-    <xacro:arg name="reverse_ip" default="0.0.0.0"/>
-    <xacro:arg name="script_command_port" default="50004"/>
-    <xacro:arg name="reverse_port" default="50001"/>
-    <xacro:arg name="script_sender_port" default="50002"/>
-    <xacro:arg name="trajectory_port" default="50003"/>
-    <xacro:arg name="use_tool_communication" default="false"/>
-    <xacro:arg name="tool_voltage" default="0"/>
-    <xacro:arg name="tool_parity" default="0"/>
-    <xacro:arg name="tool_baud_rate" default="115200"/>
-    <xacro:arg name="tool_stop_bits" default="1"/>
-    <xacro:arg name="tool_rx_idle_chars" default="1.5"/>
-    <xacro:arg name="tool_tx_idle_chars" default="3.5"/>
-    <xacro:arg name="tool_device_name" default="/tmp/ttyUR"/>
-    <xacro:arg name="tool_tcp_port" default="54321"/>
-    <xacro:arg name="use_fake_hardware" default="true"/>
-    <xacro:arg name="fake_sensor_commands" default="false"/>
-    <xacro:arg name="sim_gazebo" default="false"/>
-    <xacro:arg name="sim_ignition" default="false"/>
-    <xacro:arg name="simulation_controllers" default=""/>
-    <xacro:arg name="non_blocking_read" default="true"/>
-    <xacro:arg name="robot_receive_timeout" default="0.04"/>
-    <xacro:arg name="generate_ros2_control" default="true"/>
-    <xacro:arg name="keep_alive_count" default="2"/>
+    <!-- properties -->
+    <!-- linear guide -->
+    <xacro:property name="length" value="1.56"/>
+    <xacro:property name="min_lim" value="0.0"/>
+    <xacro:property name="max_lim" value="1.0"/>
+    <xacro:property name="vel_lim" value="0.5"/>
+    <!-- ur -->
+    <xacro:property name="ur_type" value="ur5"/>
+    <xacro:property name="name" value="ur"/>
+    <xacro:property name="tf_prefix" value=""/>
+    <xacro:property name="joint_limit_params" value="$(find ur_linear_guide)/config/ur5/joint_limits.yaml"/>
+    <xacro:property name="kinematics_params" value="$(find ur_linear_guide)/config/ur5/default_kinematics.yaml"/>
+    <xacro:property name="physical_params" value="$(find ur_linear_guide)/config/ur5/physical_parameters.yaml"/>
+    <xacro:property name="visual_params" value="$(find ur_linear_guide)/config/ur5/visual_parameters.yaml"/>
+    <xacro:property name="initial_positions_file" value="$(find ur_linear_guide)/config/ur5/initial_positions.yaml"/>
+    <xacro:property name="generate_ros2_control" value="true"/>
+    <xacro:property name="transmission_hw_interface" value=""/>
+    <xacro:property name="safety_limits" value="false"/>
+    <xacro:property name="safety_pos_margin" value="0.15"/>
+    <xacro:property name="safety_k_position" value="20"/>
+    <xacro:property name="headless_mode" value="false"/>
+    <xacro:property name="robot_ip" value="0.0.0.0"/>
+    <xacro:property name="script_filename" value=""/>
+    <xacro:property name="output_recipe_filename" value=""/>
+    <xacro:property name="input_recipe_filename" value=""/>
+    <xacro:property name="reverse_ip" value="0.0.0.0"/>
+    <xacro:property name="script_command_port" value="50004"/>
+    <xacro:property name="reverse_port" value="50001"/>
+    <xacro:property name="script_sender_port" value="50002"/>
+    <xacro:property name="trajectory_port" value="50003"/>
+    <xacro:property name="use_tool_communication" value="false"/>
+    <xacro:property name="tool_voltage" value="0"/>
+    <xacro:property name="tool_parity" value="0"/>
+    <xacro:property name="tool_baud_rate" value="115200"/>
+    <xacro:property name="tool_stop_bits" value="1"/>
+    <xacro:property name="tool_rx_idle_chars" value="1.5"/>
+    <xacro:property name="tool_tx_idle_chars" value="3.5"/>
+    <xacro:property name="tool_device_name" value="/tmp/ttyUR"/>
+    <xacro:property name="tool_tcp_port" value="54321"/>
+    <xacro:property name="fake_sensor_commands" value="false"/>
+    <xacro:property name="sim_gazebo" value="false"/>
+    <xacro:property name="sim_ignition" value="false"/>
+    <xacro:property name="simulation_controllers" value=""/>
+    <xacro:property name="non_blocking_read" value="true"/>
+    <xacro:property name="robot_receive_timeout" value="0.04"/>
+    <xacro:property name="keep_alive_count" value="2"/>
    <link name="world" />
    <!-- ur robot on linear guide -->
@@ -54,45 +57,45 @@
       fake_ur="$(arg fake_ur)"
       parent_link="world"
-      length="$(arg length)"
-      min_lim="$(arg min_lim)"
-      max_lim="$(arg max_lim)"
-      vel_lim="$(arg vel_lim)"
-      ur_type="$(arg ur_type)"
-      name="$(arg name)"
-      tf_prefix="$(arg tf_prefix)"
-      joint_limits_parameters_file="$(arg joint_limit_params)"
-      kinematics_parameters_file="$(arg kinematics_params)"
-      physical_parameters_file="$(arg physical_params)"
-      visual_parameters_file="$(arg visual_params)"
-      safety_limits="$(arg safety_limits)"
-      safety_pos_margin="$(arg safety_pos_margin)"
-      safety_k_position="$(arg safety_k_position)"
-      generate_ros2_control_tag="$(arg generate_ros2_control)"
-      transmission_hw_interface="$(arg transmission_hw_interface)"
-      fake_sensor_commands="$(arg fake_sensor_commands)"
-      sim_gazebo="$(arg sim_gazebo)"
-      sim_ignition="$(arg sim_ignition)"
-      headless_mode="$(arg headless_mode)"
-      initial_positions="$(arg initial_positions_file)"
-      use_tool_communication="$(arg use_tool_communication)"
-      tool_voltage="$(arg tool_voltage)"
-      tool_parity="$(arg tool_parity)"
-      tool_baud_rate="$(arg tool_baud_rate)"
-      tool_stop_bits="$(arg tool_stop_bits)"
-      tool_rx_idle_chars="$(arg tool_rx_idle_chars)"
-      tool_tx_idle_chars="$(arg tool_tx_idle_chars)"
-      tool_device_name="$(arg tool_device_name)"
-      tool_tcp_port="$(arg tool_tcp_port)"
-      robot_ip="$(arg robot_ip)"
-      script_filename="$(arg script_filename)"
-      output_recipe_filename="$(arg output_recipe_filename)"
-      input_recipe_filename="$(arg input_recipe_filename)"
-      reverse_port="$(arg reverse_port)"
-      script_sender_port="$(arg script_sender_port)"
-      reverse_ip="$(arg reverse_ip)"
-      script_command_port="$(arg script_command_port)"
-      trajectory_port="$(arg trajectory_port)"
-      non_blocking_read="$(arg non_blocking_read)"
-      keep_alive_count="$(arg keep_alive_count)"
+      length="${length}"
+      min_lim="${min_lim}"
+      max_lim="${max_lim}"
+      vel_lim="${vel_lim}"
+      ur_type="${ur_type}"
+      name="${name}"
+      tf_prefix="${tf_prefix}"
+      joint_limits_parameters_file="${joint_limit_params}"
+      kinematics_parameters_file="${kinematics_params}"
+      physical_parameters_file="${physical_params}"
+      visual_parameters_file="${visual_params}"
+      safety_limits="${safety_limits}"
+      safety_pos_margin="${safety_pos_margin}"
+      safety_k_position="${safety_k_position}"
+      generate_ros2_control_tag="${generate_ros2_control}"
+      transmission_hw_interface="${transmission_hw_interface}"
+      fake_sensor_commands="${fake_sensor_commands}"
+      sim_gazebo="${sim_gazebo}"
+      sim_ignition="${sim_ignition}"
+      headless_mode="${headless_mode}"
+      initial_positions="${initial_positions_file}"
+      use_tool_communication="${use_tool_communication}"
+      tool_voltage="${tool_voltage}"
+      tool_parity="${tool_parity}"
+      tool_baud_rate="${tool_baud_rate}"
+      tool_stop_bits="${tool_stop_bits}"
+      tool_rx_idle_chars="${tool_rx_idle_chars}"
+      tool_tx_idle_chars="${tool_tx_idle_chars}"
+      tool_device_name="${tool_device_name}"
+      tool_tcp_port="${tool_tcp_port}"
+      robot_ip="${robot_ip}"
+      script_filename="${script_filename}"
+      output_recipe_filename="${output_recipe_filename}"
+      input_recipe_filename="${input_recipe_filename}"
+      reverse_port="${reverse_port}"
+      script_sender_port="${script_sender_port}"
+      reverse_ip="${reverse_ip}"
+      script_command_port="${script_command_port}"
+      trajectory_port="${trajectory_port}"
+      non_blocking_read="${non_blocking_read}"
+      keep_alive_count="${keep_alive_count}"
     />
 </robot>

File: ur_linear_guide/urdf/linear_ur.xacro (robot description, xacro)
@@ -7,5 +7,5 @@
     length:=1.56
     min_lim:=0.05
-    max_lim:=1.50
+    max_lim:=1.0
     vel_lim:=0.5
     ur_type:=ur5

Commit message: wip

File: ur_linear_guide/urdf/linear_guide.xacro (robot description, xacro)
@@ -5,5 +5,5 @@
   min_lim:=0.05
   max_lim:=1.0
-  vel_lim:=0.5
+  vel_lim:=1.0
   fake_hardware:=true
 ">

File: ur_linear_guide/urdf/linear_ur.urdf.xacro (robot description, xacro)
@@ -10,5 +10,5 @@
     <xacro:property name="min_lim" value="0.0"/>
     <xacro:property name="max_lim" value="1.0"/>
-    <xacro:property name="vel_lim" value="0.5"/>
+    <xacro:property name="vel_lim" value="1.0"/>
     <!-- ur -->
     <xacro:property name="ur_type" value="ur5"/>

File: ur_linear_guide/urdf/linear_ur.xacro (robot description, xacro)
@@ -8,5 +8,5 @@
     min_lim:=0.05
     max_lim:=1.0
-    vel_lim:=0.5
+    vel_lim:=1.0
     ur_type:=ur5
     name:=ur5

Commit message: ready for plenary meeting

File: ur_linear_guide/urdf/linear_guide.xacro (robot description, xacro)
@@ -14,4 +14,7 @@
         <box size="${length} 0.1 0.1"/>
       </geometry>
+      <material name="light_grey">
+        <color rgba="0.8 0.8 0.8 1"/>
+      </material>
     </visual>
     <collision>
@@ -30,4 +33,7 @@
         <box size="0.2 0.2 0.2"/>
       </geometry>
+      <material name="light_grey">
+        <color rgba="0.8 0.8 0.8 1"/>
+      </material>
     </visual>
     <collision>

File: ur_linear_guide/urdf/linear_ur.urdf.xacro (robot description, xacro)
@@ -105,3 +105,70 @@
       <origin xyz="0 0 0" rpy="0 0 0" />
   </xacro:robotiq_gripper>
+  <!-- obstacles -->
+<link name="obstacle_cube">
+  <visual>
+    <origin xyz="0.0 0.0 0.0" rpy="0 0 0"/>
+    <geometry>
+      <box size="0.7 0.5 0.5"/>
+    </geometry>
+    <material name="grey">
+      <color rgba="0.5 0.5 0.5 1"/>
+    </material>
+  </visual>
+  <collision>
+    <origin xyz="0.0 0.0 0.0" rpy="0 0 0"/>
+    <geometry>
+      <box size="0.7 0.5 0.5"/>
+    </geometry>
+  </collision>
+</link>
+<joint name="obstacle_cube_joint" type="fixed">
+  <parent link="world"/>
+  <child link="obstacle_cube"/>
+  <origin xyz="-0.7 -0.50 -0.2" rpy="0 0 0"/>
+</joint>
+<link name="obstacle_pillar">
+  <visual>
+    <origin xyz="0.0 0.0 0.0" rpy="0 0 0"/>
+    <geometry>
+      <box size="0.1 0.1 2.0"/>
+    </geometry>
+    <material name="dark_grey">
+      <color rgba="0.2 0.2 0.2 1"/>
+    </material>
+  </visual>
+  <collision>
+    <origin xyz="0.0 0.0 0.0" rpy="0 0 0"/>
+    <geometry>
+      <box size="0.1 0.1 2.0"/>
+    </geometry>
+  </collision>
+</link>
+<joint name="obstacle_pillar_joint" type="fixed">
+  <parent link="world"/>
+  <child link="obstacle_pillar"/>
+  <origin xyz="0.80 0.25 0.5" rpy="0 0 0"/>
+</joint>
+<link name="obstacle_platform">
+  <visual>
+    <origin xyz="0.0 0.0 0.0" rpy="0 0 1.57"/>
+    <geometry>
+      <box size="1.5 0.5 0.1"/>
+    </geometry>
+    <material name="brown">
+      <color rgba="0.55 0.27 0.07 1"/>
+    </material>
+  </visual>
+  <collision>
+    <origin xyz="0.0 0.0 0.0" rpy="0 0 1.57"/>
+    <geometry>
+      <box size="1.5 0.5 0.1"/>
+    </geometry>
+  </collision>
+</link>
+<joint name="obstacle_platform_joint" type="fixed">
+  <parent link="world"/>
+  <child link="obstacle_platform"/>
+  <origin xyz="1.5 -0.65 0.0" rpy="0 0 0"/>
+</joint>
 </robot>
